File: maestro-adapter/maestro-adapter.sch (KiCad schematic (older format))
At the start: 17 parts, among them P1 CONN_01X07, P10 CONN_01X03, P11 CONN_01X03, P12 CONN_01X03, P13 CONN_01X03, P14 CONN_01X06, P15 CONN_01X06, P2 CONN_01X03, P3 CONN_01X03, P4 CONN_01X03, P5 CONN_01X03, P6 CONN_01X03, P7 CONN_01X03, P8 CONN_01X03, P9 CONN_01X03, U1 Si866x, U2 Si866x

Commit message: Update of Maestro Adapter post corrections for OSH Park Order
Parts:
- added P16: CONN_01X03, Pin_Headers:Pin_Header_Straight_1x03, symbol CONN_01X03
- added R1, R10, R11, R12, R13, R14, R15, R16, R2, R3, R4, R5, R6, R7, R8, R9: 0, Resistors_SMD:R_0603_HandSoldering, symbol R
- added W1, W10, W11, W12, W2, W3, W4, W5, W6, W7, W8, W9: TEST_1P, Measurement_Points:Measurement_Point_Round-TH_Small, symbol TEST_1P
Connections:
- net labels added: sig1_in, sig2_in, sig3_in, sig4_in, sig5_in, sig6_in, sig7_in, sig8_in, t1, t2, t3, t4
- wire segments 75 -> 139
Other:
- note added: "Power\nConnector"
- note added: "Solder bridge connections\nmust be shorted to mux inputs\nfor the input signals to be\ntransmitted."
- note added: "Solder bridges can be used to short\nover different signals to different \ninputs on the isolators. This is for\npotential faults within the maestro."
- note added: "Test Points"
- moved on the sheet: P7, P9

Commit message: Cleaned up and organized Maestro Adapter schematic
Parts:
- P16: part number (none) -> S7036-ND
Connections:
- no-connect marks 8 -> 13
Other:
- note added: "Case #1"
- note added: "Case #2"
- note added: "Maestro Connections"
- note added: "Note: tx signals are\n unused maestro \n PWM connections."
- note added: "Signal Isolators"
- note added: "Solder Bridges"
- note added: "This section intentionally left blank."
- note added: "Thruster Case\nCable Bundles"
- note added: "Thruster\nSignals 1-4"
- note added: "Thruster\nSignals 5-8"
- note added: "Thruster\nSignals 9-12"
- note removed: "Output Signal Isolators"
- note removed: "Thruster Case #1\nCable Bundle"
- note removed: "Thruster Case #2\nCable Bundle"
- note removed: "Thruster\nCase #1"
- note removed: "Thruster\nCase #2"
- note removed: "Unused\nConnections"
- moved on the sheet: P1, P10, P11, P12, P13, P14, P15, P16, P2, P3, P4, P5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
