File: pressuretester/interferenceconverterplugin.kicad_pcb (KiCad board)
At the start: 2 copper layers, 61 x 38.1 mm, 6 parts, among them P1 Mezzanine-Header, P2 CONN_02X06, U1 3mm-support, U2 3mm-support, U3 3mm-support, U4 3mm-support

Commit message: second eddition of presure tester
Routing:
- net /GND: track 0.00 -> 34.2 mm, vias 0 -> 2
- net /DTR: track 0.00 -> 25.0 mm, vias 0 -> 2
- net /CS: track 0.00 -> 24.9 mm, vias 0 -> 2
- net /AC5: track 0.00 -> 24.5 mm, vias 0 -> 2
- net /AC4: track 0.00 -> 23.5 mm, vias 0 -> 2
- net /AC3: track 0.00 -> 22.0 mm
- net /SDI: track 10.1 -> 32.0 mm, vias 1 -> 0
- net /Vbus: track 35.9 -> 29.7 mm, vias 4 -> 2
- net /TX/SCK: track 36.9 -> 36.0 mm
