File: lipo-charger/atmega1284p.sch (KiCad schematic (older format))
At the start: 15 parts

Commit message: Need to figure out mosfets
Parts:
- D? (x2): symbol LED -> LED-RESCUE-LiPoCharger
Changed lines of the file:
@@
 Place decoupling capacitors \nas close to power inputs \non microcontroller as possible.
 $Comp
-L LED D?
+L LED-RESCUE-LiPoCharger D?
 U 1 1 58268390
 P 8150 3200
@@
 DBG_LED
 $Comp
-L LED D?
+L LED-RESCUE-LiPoCharger D?
 U 1 1 58268C6C
 P 8850 3150
