File: demo-sumo-control/sumo_tank_control/sumo_tank_control.kicad_pcb (KiCad board)
At the start: 2 copper layers, 66.5 x 37 mm, 9 parts, among them J1 Conn_01x06, SW1 SW_Push, SW2 SW_Push, SW3 SW_Push, SW4 SW_Push

Commit message: Added the last two changes made to the project.
Routing:
- net /GPIO_2: track 32.3 -> 26.5 mm
Changed lines of the file:
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@@
   (segment (start 123.65 56.9125) (end 123.65 52.3625) (width 0.508) (layer F.Cu) (net 2))
   (segment (start 106.3 51.9) (end 112.8 51.9) (width 0.508) (layer F.Cu) (net 3))
-  (segment (start 112.8 51.9) (end 114.9 51.9) (width 0.508) (layer F.Cu) (net 3))
-  (segment (start 114.9 51.9) (end 120 57) (width 0.508) (layer F.Cu) (net 3))
-  (segment (start 120 57) (end 120 57) (width 0.508) (layer F.Cu) (net 3))
-  (via (at 120 57) (size 1.524) (drill 1.016) (layers F.Cu B.Cu) (net 3))
   (segment (start 130.15 55.4125) (end 128.65 56.9125) (width 0.508) (layer F.Cu) (net 3))
   (segment (start 130.15 42.312081) (end 130.15 53) (width 0.508) (layer F.Cu) (net 3))
@@
   (segment (start 130.15 53) (end 130.15 55.4125) (width 0.508) (layer F.Cu) (net 3))
   (via (at 130.15 53) (size 1.27) (drill 0.79375) (layers F.Cu B.Cu) (net 3))
+  (segment (start 113.799999 52.899999) (end 115.899999 52.899999) (width 0.508) (layer F.Cu) (net 3))
+  (segment (start 112.8 51.9) (end 113.799999 52.899999) (width 0.508) (layer F.Cu) (net 3))
+  (segment (start 115.899999 52.899999) (end 115.899999 52.899999) (width 0.508) (layer F.Cu) (net 3))
+  (via (at 115.899999 52.899999) (size 1.27) (drill 0.79375) (layers F.Cu B.Cu) (net 3))
   (segment (start 156.5 66.6) (end 163 66.6) (width 0.508) (layer F.Cu) (net 4))
   (segment (start 156.5 66.6) (end 156.1 66.6) (width 0.508) (layer F.Cu) (net 4))
